Commit message: Updated

File: tp_base/urdf/tp_robot.urdf (robot description, URDF)
Before this commit: robot tp_robot, 18 links, 17 joints
Links:
- removed link base_link
- added link base_underneath; visual cylinder length=0.005 radius=0.2
Joints:
- joint base_to_base_lap: parent base_link -> base_underneath
- joint base_to_base_up: parent base_link -> base_underneath
- joint base_to_laser: parent base_link -> base_underneath
- joint base_to_left_wheel: parent base_link -> base_underneath
- joint base_to_right_wheel: parent base_link -> base_underneath
- joint base_to_ver1: parent base_link -> base_underneath
- joint base_to_ver2: parent base_link -> base_underneath
- joint base_to_ver3: parent base_link -> base_underneath
- joint base_to_ver4: parent base_link -> base_underneath
- joint base_to_ver5: parent base_link -> base_underneath
- joint base_to_ver_left: parent base_link -> base_underneath
- joint base_to_ver_right: parent base_link -> base_underneath
- joint base_to_wheel_b: parent base_link -> base_underneath
- joint base_to_wheel_bar_b: parent base_link -> base_underneath
- joint base_to_wheel_bar_f: parent base_link -> base_underneath
- joint base_to_wheel_f: parent base_link -> base_underneath

Commit message: new tp_robot

File: tp_base/urdf/tp_robot.urdf (robot description, URDF)
Before this commit: robot tp_robot, 18 links, 17 joints
Joints:
- joint base_to_base_lap: origin xyz=-0.03 0 0.205 rpy=0 0 0 -> xyz=-0.03 0 0.155 rpy=0 0 0
- joint base_to_base_up: origin xyz=0 0 0.2 rpy=0 0 0 -> xyz=0 0 0.15 rpy=0 0 0
- joint base_to_laser: origin xyz=0.138 0 0.47 rpy=0 0 0 -> xyz=0.157 0 0.42 rpy=0 0 0
- joint base_to_left_wheel: origin xyz=0 -0.2 0.05 -> xyz=0 -0.2 0
- joint base_to_right_wheel: origin xyz=0 0.2 0.05 -> xyz=0 0.2 0
- joint base_to_ver1: origin xyz=0.125 -0.07 0.125 -> xyz=0.125 -0.07 0.075
- joint base_to_ver2: origin xyz=0.125 0.07 0.125 rpy=0 0 0 -> xyz=0.125 0.07 0.075 rpy=0 0 0
- joint base_to_ver3: origin xyz=-0.08 0.115 0.125 rpy=0 0 0 -> xyz=-0.08 0.115 0.075 rpy=0 0 0
- joint base_to_ver4: origin xyz=-0.08 -0.115 0.125 rpy=0 0 0 -> xyz=-0.08 -0.115 0.075 rpy=0 0 0
- joint base_to_ver5: origin xyz=-0.165 0 0.125 rpy=0 0 0 -> xyz=-0.165 0 0.075 rpy=0 0 0
- joint base_to_ver_left: origin xyz=0.138 0.045 0.335 rpy=0 0 0 -> xyz=0.157 0.045 0.285 rpy=0 0 0
- joint base_to_ver_right: origin xyz=0.138 -0.045 0.335 rpy=0 0 0 -> xyz=0.157 -0.045 0.285 rpy=0 0 0
- joint base_to_wheel_b: origin xyz=-0.13 0 0.014 rpy=0 0 0 -> xyz=-0.13 0 -0.036 rpy=0 0 0
- joint base_to_wheel_bar_b: origin xyz=-0.13 0 0.035 rpy=0 0 0 -> xyz=-0.13 0 -0.015 rpy=0 0 0
- joint base_to_wheel_bar_f: origin xyz=0.13 0 0.035 rpy=0 0 0 -> xyz=0.13 0 -0.015 rpy=0 0 0
- joint base_to_wheel_f: origin xyz=0.13 0 0.014 rpy=0 0 0 -> xyz=0.13 0 -0.036 rpy=0 0 0

Commit message: accurate tp_robot

File: tp_base/urdf/tp_robot.urdf (robot description, URDF)
Before this commit: robot tp_robot, 18 links, 17 joints
Links:
- added link bott_kinect; visual box size=0.05 0.08 0.03
- added link rect_bott; visual box size=0.07 0.145 0.003
- link base_laser: geometry visual box size=0.05 0.25 0.046
- link ver1: geometry visual cylinder length=0.111 radius=0.004
- link ver2: geometry visual cylinder length=0.111 radius=0.004
- link ver3: geometry visual cylinder length=0.111 radius=0.004
- link ver4: geometry visual cylinder length=0.111 radius=0.004
- link ver5: geometry visual cylinder length=0.111 radius=0.004
- link ver_laser_left: geometry visual cylinder length=0.282 radius=0.004
- link ver_laser_right: geometry visual cylinder length=0.282 radius=0.004
- link wheel_bar_behind: geometry visual box size=0.03 0.03 0.0721
- link wheel_bar_front_of: geometry visual box size=0.03 0.03 0.0721
- link wheel_behind: geometry visual sphere radius=0.02
- link wheel_front_of: geometry visual sphere radius=0.02
Joints:
- added joint base_to_rect_bott: type fixed, parent base_underneath, child rect_bott, origin xyz=0.157 0 0.393
- added joint kinect_to_bott: type fixed, parent base_laser, child bott_kinect, origin xyz=0 0 -0.038
- joint base_to_base_lap: origin xyz=-0.03 0 0.155 rpy=0 0 0 -> xyz=-0.03 0 0.123 rpy=0 0 0
- joint base_to_base_up: origin xyz=0 0 0.15 rpy=0 0 0 -> xyz=0 0 0.111 rpy=0 0 0
- joint base_to_laser: origin xyz=0.157 0 0.42 rpy=0 0 0 -> xyz=0.157 0 0.446 rpy=0 0 0
- joint base_to_left_wheel: origin xyz=0 -0.2 0 -> xyz=0 -0.181 -0.05
- joint base_to_right_wheel: origin xyz=0 0.2 0 -> xyz=0 0.181 -0.05
- joint base_to_ver1: origin xyz=0.125 -0.07 0.075 -> xyz=0.125 -0.07 0.0555
- joint base_to_ver2: origin xyz=0.125 0.07 0.075 rpy=0 0 0 -> xyz=0.125 0.07 0.0555 rpy=0 0 0
- joint base_to_ver3: origin xyz=-0.08 0.115 0.075 rpy=0 0 0 -> xyz=-0.08 0.115 0.0555 rpy=0 0 0
- joint base_to_ver4: origin xyz=-0.08 -0.115 0.075 rpy=0 0 0 -> xyz=-0.08 -0.115 0.0555 rpy=0 0 0
- joint base_to_ver5: origin xyz=-0.165 0 0.075 rpy=0 0 0 -> xyz=-0.165 0 0.0555 rpy=0 0 0
- joint base_to_ver_left: origin xyz=0.157 0.045 0.285 rpy=0 0 0 -> xyz=0.157 0.045 0.252 rpy=0 0 0
- joint base_to_ver_right: origin xyz=0.157 -0.045 0.285 rpy=0 0 0 -> xyz=0.157 -0.045 0.252 rpy=0 0 0
- joint base_to_wheel_b: origin xyz=-0.13 0 -0.036 rpy=0 0 0 -> xyz=-0.13 0 -0.08 rpy=0 0 0
- joint base_to_wheel_bar_b: origin xyz=-0.13 0 -0.015 rpy=0 0 0 -> xyz=-0.13 0 -0.03605 rpy=0 0 0
- joint base_to_wheel_bar_f: origin xyz=0.13 0 -0.015 rpy=0 0 0 -> xyz=0.13 0 -0.03605 rpy=0 0 0
- joint base_to_wheel_f: origin xyz=0.13 0 -0.036 rpy=0 0 0 -> xyz=0.13 0 -0.08 rpy=0 0 0

Commit message: updated 17/10

File: tp_base/urdf/tp_robot.urdf (robot description, URDF)
Before this commit: robot tp_robot, 20 links, 19 joints
Links:
- link base_laptop: mass None -> 0.0001; geometry collision box size=0.22 0.3 0.012; visual box size=0.22 0.3 0.012
- link base_laser: geometry collision box size=0.05 0.25 0.046; visual box size=0.05 0.25 0.046
- link base_underneath: mass None -> 0.0001; geometry collision cylinder length=0.005 radius=0.2; visual cylinder length=0.005 radius=0.2
- link base_up_robot: mass None -> 0.0001; geometry collision cylinder length=0.005 radius=0.2; visual cylinder length=0.005 radius=0.2
- link bott_kinect: mass None -> 0.0001; geometry collision box size=0.05 0.08 0.03; visual box size=0.05 0.08 0.03
- link left_wheel: mass None -> 0.0001; geometry collision cylinder length=0.02 radius=0.05; visual cylinder length=0.02 radius=0.05
- link rect_bott: mass None -> 0.0001; geometry collision box size=0.07 0.145 0.003; visual box size=0.07 0.145 0.003
- link right_wheel: mass None -> 0.0001; geometry collision cylinder length=0.02 radius=0.05; visual cylinder length=0.02 radius=0.05
- link screen_laptop: mass None -> 0.0001; geometry collision box size=0.22 0.3 0.012; visual box size=0.22 0.3 0.012
- link ver1: mass None -> 0.0001; geometry collision cylinder length=0.111 radius=0.004; visual cylinder length=0.111 radius=0.004
- link ver2: mass None -> 0.0001; geometry collision cylinder length=0.111 radius=0.004; visual cylinder length=0.111 radius=0.004
- link ver3: mass None -> 0.0001; geometry collision cylinder length=0.111 radius=0.004; visual cylinder length=0.111 radius=0.004
- link ver4: mass None -> 0.0001; geometry collision cylinder length=0.111 radius=0.004; visual cylinder length=0.111 radius=0.004
- link ver5: mass None -> 0.0001; geometry collision cylinder length=0.111 radius=0.004; visual cylinder length=0.111 radius=0.004
- link ver_laser_left: mass None -> 0.0001; geometry collision cylinder length=0.282 radius=0.004; visual cylinder length=0.282 radius=0.004
- link ver_laser_right: mass None -> 0.0001; geometry collision cylinder length=0.282 radius=0.004; visual cylinder length=0.282 radius=0.004
- link wheel_bar_behind: mass None -> 0.0001; geometry collision box size=0.03 0.03 0.0721; visual box size=0.03 0.03 0.0721
- link wheel_bar_front_of: mass None -> 0.0001; geometry collision box size=0.03 0.03 0.0721; visual box size=0.03 0.03 0.0721
- link wheel_behind: mass None -> 0.0001; geometry collision sphere radius=0.02; visual sphere radius=0.02
- link wheel_front_of: mass None -> 0.0001; geometry collision sphere radius=0.02; visual sphere radius=0.02
